Commit message: gazebo laser plugin working

File: urdf/urdf_tutorial_robot.xacro (robot description, xacro)
@@ -1,11 +1,13 @@
-<robot name="urdf_robot">
-  <link name="base_link" xmlns:xacro="http://ros.org/wiki/xacro">
-    <visual>
-      <geometry>
-        <box size="0.15 0.15 0.15"/>
+<robot name="urdf_robot"  xmlns:xacro="https://www.ros.org/wiki/xacro">
+  <xacro:include filename="$(find urdf_tutorial)/urdf/macro.xacro" />
+  <link name="base_link">
+    <pose>0 0 0.1 0 0 0</pose>
+    <visual>
+      <geometry>
+        <box size="0.5 0.3 0.07"/>
       </geometry>
       <origin rpy="0 0 0" xyz="0 0 0"/>
-      <material name="white">
-        <color rgba="1 1 1 1"/>
+      <material name="red">
+        <color rgba="1 0 0 1"/>
       </material>
     </visual>
@@ -13,19 +15,53 @@
       <origin rpy="0 0 0" xyz="0 0 0"/>
       <geometry>
-        <box size="0.15 0.15 0.15"/>
+        <box size="0.5 0.3 0.07"/>
       </geometry>
     </collision>
     <inertial>
       <origin rpy="0 0 0" xyz="0 0 0"/>
-      <mass value="0.1"/>
-      <inertia ixx="0.16666666666"  ixy="0"  ixz="0" iyy="0.16666666666" iyz="0" izz="0.16666666666" />
-    </inertial>
-  </link>
-  <link name="left_wheel">
-    <visual>
-      <geometry>
-        <cylinder length="0.02" radius="0.15"/>
-      </geometry>
-      <origin rpy="0 0 0" xyz="0 0 0"/>
+      <mass value="5"/>
+      <inertia ixx="0.0395416666667" ixy="0" ixz="0" iyy="0.106208333333" iyz="0" izz="0.106208333333" />
+    </inertial>
+  </link>
+  <link name="caster_wheel">
+    <visual>
+      <origin rpy=" 0 0 0" xyz="0.2 0 -0.05"/>
+      <geometry>
+        <sphere radius="0.05"/>
+      </geometry>
+    </visual>
+    <collision>
+      <origin rpy=" 0 0 0" xyz="0.35 0 -0.05"/>
+      <geometry>
+        <sphere radius="0.05"/>
+      </geometry>
+      <surface>
+        <friction>
+          <ode>
+            <mu>0</mu>
+            <mu2>0</mu2>
+            <slip1>1.0</slip1>
+            <slip2>1.0</slip2>
+          </ode>
+        </friction>
+      </surface>
+    </collision>
+    <inertial>
+      <origin rpy=" 0 0 0" xyz="0.35 0 -0.05"/>
+      <mass value="1"/>
+      <xacro:sphere_inertia mass="1" r="0.05" />
+    </inertial>
+  </link>
+  <joint name="joint_caster_wheel" type="fixed">
+    <origin xyz="0 0 0" rpy="0 0 0"/>
+    <parent link="base_link"/>
+    <child link="caster_wheel"/>
+  </joint>
+  <link name="right_wheel">
+    <visual>
+      <geometry>
+        <cylinder length="0.04" radius="0.1"/>
+      </geometry>
+      <origin rpy="0 1.5707 1.5707" xyz="0 0 0"/>
       <material name="black">
         <color rgba="0 0 0 1"/>
@@ -33,25 +69,26 @@
     </visual>
     <collision>
-      <origin rpy="0 0 0" xyz="0 0 0"/>
-      <geometry>
-        <cylinder length="0.02" radius="0.15"/>
-      </geometry>
-    </collision>
-    <inertial>
-      <origin rpy="0 0 0" xyz="0 0 0"/>
-      <mass value="0.025"/>
-      <!-- {{0.00575833, 0, 0}, {0, 0.00575833, 0}, {0, 0, 0.01125}} -->
-      <inertia ixx="0.00575833"  ixy="0"  ixz="0" iyy="0.00575833" iyz="0" izz="0.01125" />
-    </inertial>
-  </link>
-  <joint name="base_to_left_wheel" type="continuous">
-    <parent link="base_link"/>
-    <child link="left_wheel"/>
-    <origin rpy="-1.5708 0 0" xyz="0 0.1 0"/>
-    <axis xyz="0 0 1"/>
-  </joint>
-  <transmission name="left_wheel_transmission">
+      <origin rpy="0 1.5707 1.5707" xyz="0 0 0"/>
+      <geometry>
+        <cylinder length="0.04" radius="0.1"/>
+      </geometry>
+    </collision>
+    <inertial>
+      <origin rpy="0 1.5707 1.5707" xyz="0 0 0"/>
+      <mass value="0.2"/>
+      <inertia ixx="0.00052666666" ixy="0" ixz="0" iyy="0.00052666666" iyz="0" izz="0.001"/>
+    </inertial>
+  </link>
+  <joint name="base_to_right_wheel" type="continuous">
+    <parent link="base_link"/>
+    <child link="right_wheel"/>
+    <origin rpy="0 0 0" xyz="-0.05 0.15 0"/>
+    <axis rpy="0 0 0" xyz="0 1 0"/>
+    <limit effort="10000" velocity="1000"/>
+    <joint_properties damping="1.0" friction="1.0" />
+  </joint>
+  <transmission name="right_wheel_transmission">
     <type>transmission_interface/SimpleTransmission</type>
-    <joint name="base_to_left_wheel">
+    <joint name="base_to_right_wheel">
       <hardwareInterface>hardware_interface/VelocityJointInterface</hardwareInterface>
     </joint>
@@ -60,36 +97,38 @@
     </actuator>
 	</transmission>
-  <link name="right_wheel">
-    <visual>
-      <geometry>
-        <cylinder length="0.02" radius="0.15"/>
-      </geometry>
-      <origin rpy="0 0 0" xyz="0 0 0"/>
-      <material name="black">
-        <color rgba="0 0 0 1"/>
-      </material>
-    </visual>
-    <collision>
-      <origin rpy="0 0 0" xyz="0 0 0"/>
-      <geometry>
-        <cylinder length="0.02" radius="0.15"/>
-      </geometry>
-    </collision>
-    <inertial>
-      <origin rpy="0 0 0" xyz="0 0 0"/>
-      <mass value="0.025"/>
+  <link name="left_wheel">
+    <visual>
+      <geometry>
+        <cylinder length="0.04" radius="0.1"/>
+      </geometry>
+      <origin rpy="0 1.5707 1.5707" xyz="0 0 0"/>
+      <material name="yellow">
+        <color rgba="0.8 0.8 0.0 1.0"/>
+      </material>
+    </visual>
+    <collision>
+      <origin rpy="0 1.5707 1.5707" xyz="0 0 0"/>
+      <geometry>
+        <cylinder length="0.04" radius="0.1"/>
+      </geometry>
+    </collision>
+    <inertial>
+      <origin rpy="0 1.5707 1.5707" xyz="0 0 0"/>
+      <mass value="0.2"/>
       <!-- {{0.00575833, 0, 0}, {0, 0.00575833, 0}, {0, 0, 0.01125}} -->
-      <inertia ixx="0.00575833"  ixy="0"  ixz="0" iyy="0.00575833" iyz="0" izz="0.01125" />
-    </inertial>
-  </link>
-  <joint name="base_to_right_wheel" type="continuous">
-    <parent link="base_link"/>
-    <child link="right_wheel"/>
-    <origin rpy="-1.5708 0 0" xyz="0 -0.1 0"/>
-    <axis xyz="0 0 1"/>
-  </joint>
-  <transmission name="right_wheel_transmission">
+      <inertia ixx="0.00052666666" ixy="0" ixz="0" iyy="0.00052666666" iyz="0" izz="0.001"/>
+    </inertial>
+  </link>
+  <joint name="base_to_left_wheel" type="continuous">
+    <parent link="base_link"/>
+    <child link="left_wheel"/>
+    <origin rpy="0 0 0" xyz="-0.05 -0.15 0"/>
+    <axis rpy="0 0 0" xyz="0 1 0"/>
+    <limit effort="10000" velocity="1000"/>
+    <joint_properties damping="1.0" friction="1.0" />
+  </joint>
+  <transmission name="left_wheel_transmission">
     <type>transmission_interface/SimpleTransmission</type>
-    <joint name="base_to_right_wheel">
+    <joint name="base_to_left_wheel">
       <hardwareInterface>hardware_interface/VelocityJointInterface</hardwareInterface>
     </joint>
@@ -98,4 +137,40 @@
     </actuator>
 	</transmission>
+   <link name="sensor_laser">
+    <inertial>
+      <origin xyz="0 0 0" rpy="0 0 0" />
+      <mass value="1" />
+      <xacro:cylinder_inertia mass="1" r="0.05" l="0.1" />
+    </inertial>
+    <visual>
+      <origin xyz="0 0 0" rpy="0 0 0" />
+      <geometry>
+        <cylinder radius="0.05" length="0.1"/>
+      </geometry>
+      <material name="white">
+        <color rgba="1 1 1 1"/>
+      </material>
+    </visual>
+    <collision>
+      <origin xyz="0 0 0" rpy="0 0 0"/>
+      <geometry>
+        <cylinder radius="0.05" length="0.1"/>
+      </geometry>
+    </collision>
+  </link>
+  <joint name="joint_sensor_laser" type="fixed">
+    <origin xyz="0.15 0 0.05" rpy="0 0 0"/>
+    <parent link="base_link"/>
+    <child link="sensor_laser"/>
+  </joint>
+  <gazebo reference="base_link">
+    <material>Gazebo/Red</material>
+  </gazebo>
+  <gazebo reference="caster_wheel">
+    <material>Gazebo/Red</material>
+  </gazebo>
+  <gazebo reference="sensor_laser">
+    <material>Gazebo/White</material>
+  </gazebo>
   <gazebo reference="right_wheel">
     <mu1 value="100000.0"/>
@@ -105,4 +180,5 @@
     <fdir1 value="1 0 0"/>
     <turnGravityOff>false</turnGravityOff>
+    <material>Gazebo/Yellow</material>
   </gazebo>
   <gazebo reference="left_wheel">
@@ -113,27 +189,59 @@
     <fdir1 value="1 0 0"/>
     <turnGravityOff>false</turnGravityOff>
-  </gazebo>
-  <!-- <gazebo>
+    <material>Gazebo/Black</material>
+  </gazebo>
+  <gazebo>
     <plugin name="gazebo_ros_control" filename="libgazebo_ros_diff_drive.so">
       <robotNamespace>/</robotNamespace>
       <legacyModeNS>true</legacyModeNS>
       <alwaysOn>true</alwaysOn>
-    <legacyMode>false</legacyMode>
-    <updateRate>40</updateRate>
-    <leftJoint>base_to_left_wheel</leftJoint>
-    <rightJoint>base_to_right_wheel</rightJoint>
-    <wheelSeparation>0.2</wheelSeparation>
-    <wheelDiameter>0.15</wheelDiameter>
-    <torque>20</torque>
-    <commandTopic>cmd_vel</commandTopic>
-    <odometryTopic>odom</odometryTopic>
-    <odometryFrame>odom</odometryFrame>
-    <publishWheelTF>true</publishWheelTF>
-    <publishOdomTF>true</publishOdomTF>
-    <publishWheelJointState>true</publishWheelJointState>
-    <robotBaseFrame>base_link</robotBaseFrame>
+      <legacyMode>false</legacyMode>
+      <updateRate>40</updateRate>
+      <leftJoint>base_to_left_wheel</leftJoint>
+      <rightJoint>base_to_right_wheel</rightJoint>
+      <wheelSeparation>0.4</wheelSeparation>
+      <wheelDiameter>0.2</wheelDiameter>
+      <torque>20</torque>
+      <commandTopic>cmd_vel</commandTopic>
+      <odometryTopic>odom</odometryTopic>
+      <odometryFrame>odom</odometryFrame>
+      <publishWheelTF>true</publishWheelTF>
+      <publishOdomTF>true</publishOdomTF>
+      <publishWheelJointState>true</publishWheelJointState>
+      <robotBaseFrame>base_link</robotBaseFrame>
     </plugin>
-  </gazebo> -->
-  <gazebo>
+  </gazebo>
+  <gazebo reference="sensor_laser">
+    <sensor type="ray" name="head_hokuyo_sensor">
+      <pose>0 0 0 0 0 0</pose>
+      <visualize>false</visualize>
+      <update_rate>20</update_rate>
+      <ray>
+        <scan>
+          <horizontal>
+            <samples>720</samples>
+            <resolution>1</resolution>
+            <min_angle>-1.570796</min_angle>
+            <max_angle>1.570796</max_angle>
+          </horizontal>
+        </scan>
+        <range>
+          <min>0.10</min>
+          <max>10.0</max>
+          <resolution>0.01</resolution>
+        </range>
+        <noise>
+          <type>gaussian</type>
+          <mean>0.0</mean>
+          <stddev>0.01</stddev>
+        </noise>
+      </ray>
+      <plugin name="gazebo_ros_head_hokuyo_controller" filename="libgazebo_ros_laser.so">
+        <topicName>/laser/scan</topicName>
+        <frameName>sensor_laser</frameName>
+      </plugin>
+    </sensor>
+  </gazebo>
+  <!-- <gazebo>
     <plugin name="gazebo_ros_control" filename="libgazebo_ros_control.so">
       <robotNamespace>/</robotNamespace>
@@ -141,4 +249,4 @@
       <legacyMode>false</legacyMode>
     </plugin>
-  </gazebo>
+  </gazebo> -->
 </robot>
